File: hardware/tracker_pcb/motor.kicad_sch (KiCad schematic)
At the start: 5 parts, among them IC1 DRV8244SQRYJRQ1

Commit message: Beef up 5v supply and add new power mux
Parts:
- renumbered C10 to C13, C11 to C14, C12 to C15, C13 to C16, IC1 to U6
Changed lines of the file:
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@@
 		(dnp no)
 		(fields_autoplaced yes)
-		(property "Reference" "C11"
+		(property "Reference" "C14"
 			(at 177.8 44.8309 0)
 			(effects
@@
 			(project "tracker_pcb"
 				(path "/6aaa9514-f94e-4843-90d0-16960e4e49cb/7a9ac5e6-2be9-4d8c-8c5b-8ceb68264255"
-					(reference "C11")
+					(reference "C14")
 					(unit 1)
 				)
 				(path "/6aaa9514-f94e-4843-90d0-16960e4e49cb/f8a23924-a799-4920-a190-8ed5e6a03d20"
-					(reference "C15")
+					(reference "C18")
 					(unit 1)
 				)
@@
 		(dnp no)
 		(fields_autoplaced yes)
-		(property "Reference" "#PWR012"
+		(property "Reference" "#PWR014"
 			(at 213.36 82.55 0)
 			(effects
@@
 			(project "tracker_pcb"
 				(path "/6aaa9514-f94e-4843-90d0-16960e4e49cb/7a9ac5e6-2be9-4d8c-8c5b-8ceb68264255"
-					(reference "#PWR012")
+					(reference "#PWR014")
 					(unit 1)
 				)
 				(path "/6aaa9514-f94e-4843-90d0-16960e4e49cb/f8a23924-a799-4920-a190-8ed5e6a03d20"
-					(reference "#PWR013")
+					(reference "#PWR015")
 					(unit 1)
 				)
@@
 		(on_board yes)
 		(dnp no)
-		(property "Reference" "C13"
+		(property "Reference" "C16"
 			(at 254.254 45.72 0)
 			(effects
@@
 			(project "tracker_pcb"
 				(path "/6aaa9514-f94e-4843-90d0-16960e4e49cb/7a9ac5e6-2be9-4d8c-8c5b-8ceb68264255"
-					(reference "C13")
+					(reference "C16")
 					(unit 1)
 				)
 				(path "/6aaa9514-f94e-4843-90d0-16960e4e49cb/f8a23924-a799-4920-a190-8ed5e6a03d20"
-					(reference "C17")
+					(reference "C20")
 					(unit 1)
 				)
@@
 		(dnp no)
 		(fields_autoplaced yes)
-		(property "Reference" "IC1"
+		(property "Reference" "U6"
 			(at 215.5033 31.75 0)
 			(effects
@@
 			(project ""
 				(path "/6aaa9514-f94e-4843-90d0-16960e4e49cb/7a9ac5e6-2be9-4d8c-8c5b-8ceb68264255"
-					(reference "IC1")
+					(reference "U6")
 					(unit 1)
 				)
 				(path "/6aaa9514-f94e-4843-90d0-16960e4e49cb/f8a23924-a799-4920-a190-8ed5e6a03d20"
-					(reference "IC2")
+					(reference "U7")
 					(unit 1)
 				)
@@
 		(on_board yes)
 		(dnp no)
-		(property "Reference" "C12"
+		(property "Reference" "C15"
 			(at 240.284 45.974 0)
 			(effects
@@
 			(project "tracker_pcb"
 				(path "/6aaa9514-f94e-4843-90d0-16960e4e49cb/7a9ac5e6-2be9-4d8c-8c5b-8ceb68264255"
-					(reference "C12")
+					(reference "C15")
 					(unit 1)
 				)
 				(path "/6aaa9514-f94e-4843-90d0-16960e4e49cb/f8a23924-a799-4920-a190-8ed5e6a03d20"
-					(reference "C16")
+					(reference "C19")
 					(unit 1)
 				)
@@
 		(on_board yes)
 		(dnp no)
-		(property "Reference" "C10"
+		(property "Reference" "C13"
 			(at 163.576 44.958 0)
 			(effects
@@
 			(project "tracker_pcb"
 				(path "/6aaa9514-f94e-4843-90d0-16960e4e49cb/7a9ac5e6-2be9-4d8c-8c5b-8ceb68264255"
-					(reference "C10")
+					(reference "C13")
 					(unit 1)
 				)
 				(path "/6aaa9514-f94e-4843-90d0-16960e4e49cb/f8a23924-a799-4920-a190-8ed5e6a03d20"
-					(reference "C14")
-					(unit 1)
-				)
+					(reference "C17")
+					(unit 1)
+				)

Commit message: Modify iso circuit for best CTR
Parts:
- U6: footprint DRV8244HQRYJRQ1 -> footprint:DRV8244HQRYJRQ1
- renumbered C13 to C12, C14 to C13, C15 to C14, C16 to C15
Changed lines of the file:
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@@
 		(dnp no)
 		(fields_autoplaced yes)
-		(property "Reference" "C14"
+		(property "Reference" "C13"
 			(at 177.8 44.8309 0)
 			(effects
@@
 			(project "tracker_pcb"
 				(path "/6aaa9514-f94e-4843-90d0-16960e4e49cb/7a9ac5e6-2be9-4d8c-8c5b-8ceb68264255"
-					(reference "C14")
+					(reference "C13")
 					(unit 1)
 				)
 				(path "/6aaa9514-f94e-4843-90d0-16960e4e49cb/f8a23924-a799-4920-a190-8ed5e6a03d20"
-					(reference "C18")
+					(reference "C17")
 					(unit 1)
 				)
@@
 		(on_board yes)
 		(dnp no)
-		(property "Reference" "C16"
+		(property "Reference" "C15"
 			(at 254.254 45.72 0)
 			(effects
@@
 			(project "tracker_pcb"
 				(path "/6aaa9514-f94e-4843-90d0-16960e4e49cb/7a9ac5e6-2be9-4d8c-8c5b-8ceb68264255"
-					(reference "C16")
+					(reference "C15")
 					(unit 1)
 				)
 				(path "/6aaa9514-f94e-4843-90d0-16960e4e49cb/f8a23924-a799-4920-a190-8ed5e6a03d20"
-					(reference "C20")
+					(reference "C19")
 					(unit 1)
 				)
@@
 			)
 		)
-		(property "Footprint" "DRV8244HQRYJRQ1"
+		(property "Footprint" "footprint:DRV8244HQRYJRQ1"
 			(at 226.06 134.29 0)
 			(effects
@@
 		(on_board yes)
 		(dnp no)
-		(property "Reference" "C15"
+		(property "Reference" "C14"
 			(at 240.284 45.974 0)
 			(effects
@@
 			(project "tracker_pcb"
 				(path "/6aaa9514-f94e-4843-90d0-16960e4e49cb/7a9ac5e6-2be9-4d8c-8c5b-8ceb68264255"
-					(reference "C15")
+					(reference "C14")
 					(unit 1)
 				)
 				(path "/6aaa9514-f94e-4843-90d0-16960e4e49cb/f8a23924-a799-4920-a190-8ed5e6a03d20"
-					(reference "C19")
+					(reference "C18")
 					(unit 1)
 				)
@@
 		(on_board yes)
 		(dnp no)
-		(property "Reference" "C13"
+		(property "Reference" "C12"
 			(at 163.576 44.958 0)
 			(effects
@@
 			(project "tracker_pcb"
 				(path "/6aaa9514-f94e-4843-90d0-16960e4e49cb/7a9ac5e6-2be9-4d8c-8c5b-8ceb68264255"
-					(reference "C13")
+					(reference "C12")
 					(unit 1)
 				)
 				(path "/6aaa9514-f94e-4843-90d0-16960e4e49cb/f8a23924-a799-4920-a190-8ed5e6a03d20"
-					(reference "C17")
-					(unit 1)
-				)
+					(reference "C16")
+					(unit 1)
+				)
