File: hardware/tracker_pcb/motor.kicad_sch (KiCad schematic)
At the start: 5 parts, among them U6 DRV8244SQRYJRQ1

Commit message: v2 hardware changes
Parts:
- added D4: SMBJ30CA, PCM_JLCPCB:D_SMB, symbol PCM_JLCPCB-Diodes:TVS-Bi,SMBJ30CA
- C14: renamed from C13; footprint Capacitor_SMD:CP_Elec_10x12.5 -> Capacitor_SMD:CP_Elec_18x17.5
- renumbered C12 to C13, C14 to C15, C15 to C16
Connections:
- net OUT1: now also D4.2
- net OUT2: now also D4.1

Commit message: more motor safety
Parts:
- renumbered C13 to C12, C14 to C13, C15 to C14, C16 to C15, U6 to U4
Connections:
- net GND: no longer U4.10 (DRVOFF)
- new net DRVOFF: U4.10 (DRVOFF)
Changed lines of the file:
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@@
 		(color 0 0 0 0)
 	)
-	(junction
-		(at 241.3 72.39)
-		(diameter 0)
-		(color 0 0 0 0)
-	)
 	(wire
 		(pts
@@
 	(wire
 		(pts
-			(xy 241.3 72.39) (xy 246.38 72.39)
+			(xy 229.87 49.53) (xy 231.14 49.53)
 		)
 		(stroke
@@
 	(wire
 		(pts
-			(xy 229.87 49.53) (xy 241.3 49.53)
-		)
-		(stroke
-			(width 0)
-			(type default)
-		)
-	)
-	(wire
-		(pts
 			(xy 213.36 64.77) (xy 213.36 72.39)
 		)
@@
 	(wire
 		(pts
-			(xy 241.3 49.53) (xy 241.3 72.39)
-		)
-		(stroke
-			(width 0)
-			(type default)
-		)
-	)
-	(wire
-		(pts
 			(xy 232.41 40.64) (xy 246.38 40.64)
 		)
@@
 	(wire
 		(pts
-			(xy 229.87 72.39) (xy 241.3 72.39)
+			(xy 229.87 72.39) (xy 246.38 72.39)
 		)
 		(stroke
@@
 			)
 			(justify right)
+		)
+	)
+	(hierarchical_label "DRVOFF"
+		(shape input)
+		(at 231.14 49.53 0)
+		(effects
+			(font
+				(size 1.27 1.27)
+			)
+			(justify left)
 		)
 	)
@@
 		(dnp no)
 		(fields_autoplaced yes)
-		(property "Reference" "C14"
+		(property "Reference" "C13"
 			(at 177.8 44.8309 0)
 			(effects
@@
 			(project "tracker_pcb"
 				(path "/6aaa9514-f94e-4843-90d0-16960e4e49cb/7a9ac5e6-2be9-4d8c-8c5b-8ceb68264255"
-					(reference "C14")
+					(reference "C13")
 					(unit 1)
 				)
 				(path "/6aaa9514-f94e-4843-90d0-16960e4e49cb/f8a23924-a799-4920-a190-8ed5e6a03d20"
-					(reference "C18")
+					(reference "C17")
 					(unit 1)
 				)
@@
 		(dnp no)
 		(fields_autoplaced yes)
-		(property "Reference" "#PWR015"
+		(property "Reference" "#PWR012"
 			(at 213.36 82.55 0)
 			(effects
@@
 			(project "tracker_pcb"
 				(path "/6aaa9514-f94e-4843-90d0-16960e4e49cb/7a9ac5e6-2be9-4d8c-8c5b-8ceb68264255"
-					(reference "#PWR015")
+					(reference "#PWR012")
 					(unit 1)
 				)
 				(path "/6aaa9514-f94e-4843-90d0-16960e4e49cb/f8a23924-a799-4920-a190-8ed5e6a03d20"
-					(reference "#PWR016")
+					(reference "#PWR013")
 					(unit 1)
 				)
@@
 		(on_board yes)
 		(dnp no)
-		(property "Reference" "C16"
+		(property "Reference" "C15"
 			(at 254.254 45.72 0)
 			(effects
@@
 			(project "tracker_pcb"
 				(path "/6aaa9514-f94e-4843-90d0-16960e4e49cb/7a9ac5e6-2be9-4d8c-8c5b-8ceb68264255"
-					(reference "C16")
+					(reference "C15")
 					(unit 1)
 				)
 				(path "/6aaa9514-f94e-4843-90d0-16960e4e49cb/f8a23924-a799-4920-a190-8ed5e6a03d20"
-					(reference "C20")
+					(reference "C19")
 					(unit 1)
 				)
@@
 		(on_board yes)
 		(dnp no)
-		(property "Reference" "U6"
+		(property "Reference" "U4"
 			(at 192.532 59.436 0)
 			(effects
@@
 			(project ""
 				(path "/6aaa9514-f94e-4843-90d0-16960e4e49cb/7a9ac5e6-2be9-4d8c-8c5b-8ceb68264255"
-					(reference "U6")
+					(reference "U4")
 					(unit 1)
 				)
 				(path "/6aaa9514-f94e-4843-90d0-16960e4e49cb/f8a23924-a799-4920-a190-8ed5e6a03d20"
-					(reference "U7")
+					(reference "U5")
 					(unit 1)
 				)
@@
 		(on_board yes)
 		(dnp no)
-		(property "Reference" "C15"
+		(property "Reference" "C14"
 			(at 240.284 45.974 0)
 			(effects
@@
 			(project "tracker_pcb"
 				(path "/6aaa9514-f94e-4843-90d0-16960e4e49cb/7a9ac5e6-2be9-4d8c-8c5b-8ceb68264255"
-					(reference "C15")
+					(reference "C14")
 					(unit 1)
 				)
 				(path "/6aaa9514-f94e-4843-90d0-16960e4e49cb/f8a23924-a799-4920-a190-8ed5e6a03d20"
-					(reference "C19")
+					(reference "C18")
 					(unit 1)
 				)
@@
 		(on_board yes)
 		(dnp no)
-		(property "Reference" "C13"
+		(property "Reference" "C12"
 			(at 163.576 44.958 0)
 			(effects
@@
 			(project "tracker_pcb"
 				(path "/6aaa9514-f94e-4843-90d0-16960e4e49cb/7a9ac5e6-2be9-4d8c-8c5b-8ceb68264255"
-					(reference "C13")
+					(reference "C12")
 					(unit 1)
 				)
 				(path "/6aaa9514-f94e-4843-90d0-16960e4e49cb/f8a23924-a799-4920-a190-8ed5e6a03d20"
-					(reference "C17")
+					(reference "C16")
 					(unit 1)
 				)
