File: hardware/tracker_pcb/rs485.kicad_sch (KiCad schematic)
At the start: 6 parts, among them U8 THVD1426DRLR

Commit message: v2 hardware changes
Parts:
- renumbered C20 to C21, D4 to D6, R10 to R12, R11 to R13, R12 to R14
Changed lines of the file:
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@@
 	(wire
 		(pts
-			(xy 172.72 85.09) (xy 175.26 85.09)
+			(xy 107.95 67.31) (xy 134.62 67.31)
 		)
 		(stroke
@@
 	(wire
 		(pts
-			(xy 107.95 67.31) (xy 134.62 67.31)
+			(xy 172.72 85.09) (xy 191.77 85.09)
 		)
 		(stroke
@@
 	(wire
 		(pts
-			(xy 172.72 72.39) (xy 175.26 72.39)
+			(xy 160.02 78.74) (xy 162.56 78.74)
 		)
 		(stroke
@@
 	(wire
 		(pts
-			(xy 160.02 78.74) (xy 162.56 78.74)
+			(xy 148.59 77.47) (xy 148.59 72.39)
 		)
 		(stroke
@@
 	(wire
 		(pts
-			(xy 148.59 77.47) (xy 148.59 72.39)
+			(xy 172.72 72.39) (xy 191.77 72.39)
 		)
 		(stroke
@@
 	(hierarchical_label "B"
 		(shape passive)
-		(at 175.26 85.09 0)
+		(at 191.77 85.09 0)
 		(effects
 			(font
@@
 	(hierarchical_label "A"
 		(shape passive)
-		(at 175.26 72.39 0)
+		(at 191.77 72.39 0)
 		(effects
 			(font
@@
 		(on_board yes)
 		(dnp no)
-		(property "Reference" "D4"
+		(property "Reference" "D6"
 			(at 178.054 76.454 90)
 			(effects
@@
 			(project "tracker_pcb"
 				(path "/6aaa9514-f94e-4843-90d0-16960e4e49cb/b3bc6330-02c7-43c9-a193-56a83bf675dc"
-					(reference "D4")
+					(reference "D6")
 					(unit 1)
 				)
@@
 		(on_board yes)
 		(dnp no)
-		(property "Reference" "R10"
+		(property "Reference" "R12"
 			(at 156.464 76.454 0)
 			(effects
@@
 			(project "tracker_pcb"
 				(path "/6aaa9514-f94e-4843-90d0-16960e4e49cb/b3bc6330-02c7-43c9-a193-56a83bf675dc"
-					(reference "R10")
+					(reference "R12")
 					(unit 1)
 				)
@@
 		(dnp no)
 		(fields_autoplaced yes)
-		(property "Reference" "#PWR017"
+		(property "Reference" "#PWR018"
 			(at 160.02 85.09 0)
 			(effects
@@
 			(project "tracker_pcb"
 				(path "/6aaa9514-f94e-4843-90d0-16960e4e49cb/b3bc6330-02c7-43c9-a193-56a83bf675dc"
-					(reference "#PWR017")
+					(reference "#PWR018")
 					(unit 1)
 				)
@@
 		(on_board yes)
 		(dnp no)
-		(property "Reference" "R11"
+		(property "Reference" "R13"
 			(at 162.814 68.58 90)
 			(effects
@@
 			(project "tracker_pcb"
 				(path "/6aaa9514-f94e-4843-90d0-16960e4e49cb/b3bc6330-02c7-43c9-a193-56a83bf675dc"
-					(reference "R11")
+					(reference "R13")
 					(unit 1)
 				)
@@
 		(dnp no)
 		(fields_autoplaced yes)
-		(property "Reference" "C20"
+		(property "Reference" "C21"
 			(at 124.46 88.8999 0)
 			(effects
@@
 			(project "tracker_pcb"
 				(path "/6aaa9514-f94e-4843-90d0-16960e4e49cb/b3bc6330-02c7-43c9-a193-56a83bf675dc"
-					(reference "C20")
+					(reference "C21")
 					(unit 1)
 				)
@@
 		(on_board yes)
 		(dnp no)
-		(property "Reference" "R12"
+		(property "Reference" "R14"
 			(at 161.798 86.614 90)
 			(effects
@@
 			(project "tracker_pcb"
 				(path "/6aaa9514-f94e-4843-90d0-16960e4e49cb/b3bc6330-02c7-43c9-a193-56a83bf675dc"
-					(reference "R12")
+					(reference "R14")
 					(unit 1)
 				)
@@
 		(dnp no)
 		(fields_autoplaced yes)
-		(property "Reference" "#PWR016"
+		(property "Reference" "#PWR017"
 			(at 134.62 102.87 0)
 			(effects
@@
 			(project "tracker_pcb"
 				(path "/6aaa9514-f94e-4843-90d0-16960e4e49cb/b3bc6330-02c7-43c9-a193-56a83bf675dc"
-					(reference "#PWR016")
+					(reference "#PWR017")
 					(unit 1)
 				)

Commit message: more motor safety
Parts:
- renumbered C21 to C20, U8 to U6
Changed lines of the file:
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@@
 		(dnp no)
 		(fields_autoplaced yes)
-		(property "Reference" "#PWR018"
+		(property "Reference" "#PWR015"
 			(at 160.02 85.09 0)
 			(effects
@@
 			(project "tracker_pcb"
 				(path "/6aaa9514-f94e-4843-90d0-16960e4e49cb/b3bc6330-02c7-43c9-a193-56a83bf675dc"
-					(reference "#PWR018")
+					(reference "#PWR015")
 					(unit 1)
 				)
@@
 		(dnp no)
 		(fields_autoplaced yes)
-		(property "Reference" "C21"
+		(property "Reference" "C20"
 			(at 124.46 88.8999 0)
 			(effects
@@
 			(project "tracker_pcb"
 				(path "/6aaa9514-f94e-4843-90d0-16960e4e49cb/b3bc6330-02c7-43c9-a193-56a83bf675dc"
-					(reference "C21")
+					(reference "C20")
 					(unit 1)
 				)
@@
 		(dnp no)
 		(fields_autoplaced yes)
-		(property "Reference" "U8"
+		(property "Reference" "U6"
 			(at 136.7633 67.31 0)
 			(effects
@@
 			(project "tracker_pcb"
 				(path "/6aaa9514-f94e-4843-90d0-16960e4e49cb/b3bc6330-02c7-43c9-a193-56a83bf675dc"
-					(reference "U8")
+					(reference "U6")
 					(unit 1)
 				)
@@
 		(dnp no)
 		(fields_autoplaced yes)
-		(property "Reference" "#PWR017"
+		(property "Reference" "#PWR014"
 			(at 134.62 102.87 0)
 			(effects
@@
 			(project "tracker_pcb"
 				(path "/6aaa9514-f94e-4843-90d0-16960e4e49cb/b3bc6330-02c7-43c9-a193-56a83bf675dc"
-					(reference "#PWR017")
+					(reference "#PWR014")
 					(unit 1)
 				)
