File: hardware/tracker_pcb/ESP32-C6-MINI-1U-N4.kicad_sch (KiCad schematic)
At the start: 1 part, among them U4 ESP32-C6-MINI-1U-N4

Commit message: VIA changes
Parts:
- U4: LCSC (none) -> C22399676
Changed lines of the file:
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@@
+			)
+		)
+		(property "LCSC" "C22399676"
+			(at 119.38 33.02 0)
+			(effects
+				(font
+					(size 1.27 1.27)
+				)
+				(hide yes)
 			)
 		)

Commit message: update BOM
Parts:
- U4: LCSC C22399676 -> C485916
Changed lines of the file:
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@@
 			)
 		)
-		(property "LCSC" "C22399676"
+		(property "LCSC" "C485916"
 			(at 119.38 33.02 0)
 			(effects
