File: hardware/tracker_pcb/esp32.kicad_sch (KiCad schematic)
At the start: 17 parts, among them J4 USB_C_Receptacle_USB2.0_16P, SW1 SKRKAEE020, SW2 SKRKAEE020, U1 USBLC6-2SC6, U6 ESP32-C6-MINI-1U-N4, U7 SN74LVC1G139

Commit message: VIA changes
Parts:
- C19: LCSC (none) -> C1591
- C20: LCSC (none) -> C1644
- J4: LCSC (none) -> C5184243
- R20, R21, R26: LCSC (none) -> C23186
- R22, R23: LCSC (none) -> C23345
- R24, R25: LCSC (none) -> C25804
- SW1, SW2: LCSC (none) -> C115357
- U1: LCSC (none) -> C7519
- U6: LCSC (none) -> C20627095
- U7: LCSC (none) -> C2653305
Changed lines of the file:
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@@
+			)
+		)
+		(property "LCSC" "C23345"
+			(at 88.646 85.344 0)
+			(effects
+				(font
+					(size 1.27 1.27)
+				)
+				(hide yes)
 			)
 		)
@@
 			)
 		)
+		(property "LCSC" "C23345"
+			(at 88.646 80.264 0)
+			(effects
+				(font
+					(size 1.27 1.27)
+				)
+				(hide yes)
+			)
+		)
 		(pin "1"
 		)
@@
 		(property "Description" "Resistor, US symbol"
 			(at 69.85 72.39 0)
+			(effects
+				(font
+					(size 1.27 1.27)
+				)
+				(hide yes)
+			)
+		)
+		(property "LCSC" "C23186"
+			(at 65.532 70.866 0)
 			(effects
 				(font
@@
 			)
 		)
+		(property "LCSC" "C25804"
+			(at 147.32 90.1699 0)
+			(effects
+				(font
+					(size 1.27 1.27)
+				)
+				(hide yes)
+			)
+		)
 		(pin "1"
 		)
@@
 			)
 		)
+		(property "LCSC" "C20627095"
+			(at 196.85 55.88 0)
+			(effects
+				(font
+					(size 1.27 1.27)
+				)
+				(hide yes)
+			)
+		)
 		(pin "13"
 		)
@@
 			)
 		)
+		(property "LCSC" "C1591"
+			(at 143.764 74.168 0)
+			(effects
+				(font
+					(size 1.27 1.27)
+				)
+				(hide yes)
+			)
+		)
 		(pin "2"
 		)
@@
 		(property "Description" "Unpolarized capacitor"
 			(at 151.13 106.68 0)
+			(effects
+				(font
+					(size 1.27 1.27)
+				)
+				(hide yes)
+			)
+		)
+		(property "LCSC" "C1644"
+			(at 153.924 104.648 0)
 			(effects
 				(font
@@
 			)
 		)
+		(property "LCSC" "C2653305"
+			(at 130.4133 139.7 0)
+			(effects
+				(font
+					(size 1.27 1.27)
+				)
+				(hide yes)
+			)
+		)
 		(pin "D1"
 		)
@@
 		(property "Description" "Resistor, US symbol"
 			(at 69.85 68.58 0)
+			(effects
+				(font
+					(size 1.27 1.27)
+				)
+				(hide yes)
+			)
+		)
+		(property "LCSC" "C23186"
+			(at 65.532 67.056 0)
 			(effects
 				(font
@@
 			)
 		)
+		(property "LCSC" "C7519"
+			(at 81.6611 72.39 0)
+			(effects
+				(font
+					(size 1.27 1.27)
+				)
+				(hide yes)
+			)
+		)
 		(pin "3"
 		)
@@
 			)
 		)
+		(property "LCSC" "C25804"
+			(at 137.16 60.9599 0)
+			(effects
+				(font
+					(size 1.27 1.27)
+				)
+				(hide yes)
+			)
+		)
 		(pin "1"
 		)
@@
 			)
 		)
+		(property "LCSC" "C23186"
+			(at 156.21 81.28 0)
+			(effects
+				(font
+					(size 1.27 1.27)
+				)
+				(hide yes)
+			)
+		)
 		(pin "1"
 		)
@@
 			)
 		)
+		(property "LCSC" "C115357"
+			(at 130.81 73.6599 0)
+			(effects
+				(font
+					(size 1.27 1.27)
+				)
+				(hide yes)
+			)
+		)
 		(pin "1"
 		)
@@
 			)
 		)
+		(property "LCSC" "C5184243"
+			(at 46.99 55.88 0)
+			(effects
+				(font
+					(size 1.27 1.27)
+				)
+				(hide yes)
+			)
+		)
 		(pin "B4"
 		)
@@
 			(effects
 				(font
+					(size 1.27 1.27)
+				)
+				(hide yes)
+			)
+		)
+		(property "LCSC" "C115357"
+			(at 140.97 104.1399 0)
+			(effects
+				(font

Commit message: Beef up 5v supply and add new power mux
Parts:
- renumbered C1 to C22, C19 to C23, C20 to C24, C21 to C25, J4 to J7, R20 to R19, R21 to R20, R22 to R21, R23 to R22, R24 to R23, R25 to R24, R26 to R25, U7 to U10, U6 to U11, U1 to U9
Changed lines of the file:
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@@
 		(on_board yes)
 		(dnp no)
-		(property "Reference" "R23"
+		(property "Reference" "R22"
 			(at 88.646 85.344 90)
 			(effects
@@
 			(project "tracker_pcb"
 				(path "/6aaa9514-f94e-4843-90d0-16960e4e49cb/856fce88-9666-4784-b480-ab1432c6ba59"
-					(reference "R23")
+					(reference "R22")
 					(unit 1)
 				)
@@
 		(on_board yes)
 		(dnp no)
-		(property "Reference" "R22"
+		(property "Reference" "R21"
 			(at 88.646 80.264 90)
 			(effects
@@
 			(project "tracker_pcb"
 				(path "/6aaa9514-f94e-4843-90d0-16960e4e49cb/856fce88-9666-4784-b480-ab1432c6ba59"
-					(reference "R22")
+					(reference "R21")
 					(unit 1)
 				)
@@
 		(on_board yes)
 		(dnp no)
-		(property "Reference" "C21"
+		(property "Reference" "C25"
 			(at 232.664 65.278 0)
 			(effects
@@
 			(project "tracker_pcb"
 				(path "/6aaa9514-f94e-4843-90d0-16960e4e49cb/856fce88-9666-4784-b480-ab1432c6ba59"
-					(reference "C21")
+					(reference "C25")
 					(unit 1)
 				)
@@
 		(on_board yes)
 		(dnp no)
-		(property "Reference" "R21"
+		(property "Reference" "R20"
 			(at 65.532 70.866 90)
 			(effects
@@
 			(project "tracker_pcb"
 				(path "/6aaa9514-f94e-4843-90d0-16960e4e49cb/856fce88-9666-4784-b480-ab1432c6ba59"
-					(reference "R21")
+					(reference "R20")
 					(unit 1)
 				)
@@
 		(dnp no)
 		(fields_autoplaced yes)
-		(property "Reference" "#PWR020"
+		(property "Reference" "#PWR025"
 			(at 229.87 125.73 0)
 			(effects
@@
 			(project "tracker_pcb"
 				(path "/6aaa9514-f94e-4843-90d0-16960e4e49cb/856fce88-9666-4784-b480-ab1432c6ba59"
-					(reference "#PWR020")
+					(reference "#PWR025")
 					(unit 1)
 				)
@@
 		(dnp no)
 		(fields_autoplaced yes)
-		(property "Reference" "R25"
+		(property "Reference" "R24"
 			(at 147.32 90.1699 0)
 			(effects
@@
 			(project "tracker_pcb"
 				(path "/6aaa9514-f94e-4843-90d0-16960e4e49cb/856fce88-9666-4784-b480-ab1432c6ba59"
-					(reference "R25")
+					(reference "R24")
 					(unit 1)
 				)
@@
 		(on_board yes)
 		(dnp no)
-		(property "Reference" "C1"
+		(property "Reference" "C22"
 			(at 98.298 151.638 0)
 			(effects
@@
 			(project "tracker_pcb"
 				(path "/6aaa9514-f94e-4843-90d0-16960e4e49cb/856fce88-9666-4784-b480-ab1432c6ba59"
-					(reference "C1")
+					(reference "C22")
 					(unit 1)
 				)
@@
 		(dnp no)
 		(fields_autoplaced yes)
-		(property "Reference" "#PWR08"
+		(property "Reference" "#PWR023"
 			(at 80.01 109.22 0)
 			(effects
@@
 			(project "tracker_pcb"
 				(path "/6aaa9514-f94e-4843-90d0-16960e4e49cb/856fce88-9666-4784-b480-ab1432c6ba59"
-					(reference "#PWR08")
+					(reference "#PWR023")
 					(unit 1)
 				)
@@
 		(dnp no)
 		(fields_autoplaced yes)
-		(property "Reference" "U6"
+		(property "Reference" "U11"
 			(at 196.85 55.88 0)
 			(effects
@@
 			(project "tracker_pcb"
 				(path "/6aaa9514-f94e-4843-90d0-16960e4e49cb/856fce88-9666-4784-b480-ab1432c6ba59"
-					(reference "U6")
+					(reference "U11")
 					(unit 1)
 				)
@@
 		(on_board yes)
 		(dnp no)
-		(property "Reference" "C19"
+		(property "Reference" "C23"
 			(at 143.764 74.168 0)
 			(effects
@@
 			(project "tracker_pcb"
 				(path "/6aaa9514-f94e-4843-90d0-16960e4e49cb/856fce88-9666-4784-b480-ab1432c6ba59"
-					(reference "C19")
+					(reference "C23")
 					(unit 1)
 				)
@@
 		(on_board yes)
 		(dnp no)
-		(property "Reference" "C20"
+		(property "Reference" "C24"
 			(at 153.924 104.648 0)
 			(effects
@@
 			(project "tracker_pcb"
 				(path "/6aaa9514-f94e-4843-90d0-16960e4e49cb/856fce88-9666-4784-b480-ab1432c6ba59"
-					(reference "C20")
+					(reference "C24")
 					(unit 1)
 				)
@@
 		(dnp no)
 		(fields_autoplaced yes)
-		(property "Reference" "#PWR023"
+		(property "Reference" "#PWR024"
 			(at 104.14 175.26 0)
 			(effects
@@
 			(project "tracker_pcb"
 				(path "/6aaa9514-f94e-4843-90d0-16960e4e49cb/856fce88-9666-4784-b480-ab1432c6ba59"
-					(reference "#PWR023")
+					(reference "#PWR024")
 					(unit 1)
 				)
@@
 		(dnp no)
 		(fields_autoplaced yes)
-		(property "Reference" "U7"
+		(property "Reference" "U10"
 			(at 130.4133 139.7 0)
 			(effects
@@
 			(project "tracker_pcb"
 				(path "/6aaa9514-f94e-4843-90d0-16960e4e49cb/856fce88-9666-4784-b480-ab1432c6ba59"
-					(reference "U7")
+					(reference "U10")
 					(unit 1)
 				)
@@
 		(on_board yes)
 		(dnp no)
-		(property "Reference" "R20"
+		(property "Reference" "R19"
 			(at 65.532 67.056 90)
 			(effects
@@
 			(project "tracker_pcb"
 				(path "/6aaa9514-f94e-4843-90d0-16960e4e49cb/856fce88-9666-4784-b480-ab1432c6ba59"
-					(reference "R20")
+					(reference "R19")
 					(unit 1)
 				)
@@
 		(dnp no)
 		(fields_autoplaced yes)
-		(property "Reference" "#PWR021"
+		(property "Reference" "#PWR022"
 			(at 73.66 81.28 0)
 			(effects
@@
 			(project "tracker_pcb"
 				(path "/6aaa9514-f94e-4843-90d0-16960e4e49cb/856fce88-9666-4784-b480-ab1432c6ba59"
-					(reference "#PWR021")
+					(reference "#PWR022")
 					(unit 1)
 				)
@@
 		(dnp no)
 		(fields_autoplaced yes)
-		(property "Reference" "U1"
+		(property "Reference" "U9"
 			(at 81.6611 72.39 0)
 			(effects
@@
 			(project ""
 				(path "/6aaa9514-f94e-4843-90d0-16960e4e49cb/856fce88-9666-4784-b480-ab1432c6ba59"
-					(reference "U1")
+					(reference "U9")
 					(unit 1)
 				)
@@
 		(dnp no)
 		(fields_autoplaced yes)
-		(property "Reference" "R24"
+		(property "Reference" "R23"
 			(at 137.16 60.9599 0)
 			(effects
@@
 			(project "tracker_pcb"
 				(path "/6aaa9514-f94e-4843-90d0-16960e4e49cb/856fce88-9666-4784-b480-ab1432c6ba59"
-					(reference "R24")
+					(reference "R23")
 					(unit 1)
 				)
@@
 		(dnp no)
 		(fields_autoplaced yes)
-		(property "Reference" "R26"
+		(property "Reference" "R25"
 			(at 156.21 81.28 90)
 			(effects
@@
 			(project "tracker_pcb"
 				(path "/6aaa9514-f94e-4843-90d0-16960e4e49cb/856fce88-9666-4784-b480-ab1432c6ba59"
-					(reference "R26")
+					(reference "R25")
 					(unit 1)
 				)
@@
 		(dnp no)
 		(fields_autoplaced yes)
-		(property "Reference" "J4"
+		(property "Reference" "J7"
 			(at 46.99 55.88 0)
 			(effects
@@
 			(project "tracker_pcb"
 				(path "/6aaa9514-f94e-4843-90d0-16960e4e49cb/856fce88-9666-4784-b480-ab1432c6ba59"
-					(reference "J4")
-					(unit 1)
-				)
+					(reference "J7")
+					(unit 1)
+				)

Commit message: Modify iso circuit for best CTR
Parts:
- renumbered C22 to C21, C23 to C22, C24 to C23, C25 to C24, J7 to J8, R19 to R21, R20 to R22, R21 to R23, R22 to R24, R23 to R25, R24 to R26, R25 to R27
Changed lines of the file:
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@@
 		(on_board yes)
 		(dnp no)
-		(property "Reference" "R22"
+		(property "Reference" "R24"
 			(at 88.646 85.344 90)
 			(effects
@@
 			(project "tracker_pcb"
 				(path "/6aaa9514-f94e-4843-90d0-16960e4e49cb/856fce88-9666-4784-b480-ab1432c6ba59"
-					(reference "R22")
+					(reference "R24")
 					(unit 1)
 				)
@@
 		(on_board yes)
 		(dnp no)
-		(property "Reference" "R21"
+		(property "Reference" "R23"
 			(at 88.646 80.264 90)
 			(effects
@@
 			(project "tracker_pcb"
 				(path "/6aaa9514-f94e-4843-90d0-16960e4e49cb/856fce88-9666-4784-b480-ab1432c6ba59"
-					(reference "R21")
+					(reference "R23")
 					(unit 1)
 				)
@@
 		(on_board yes)
 		(dnp no)
-		(property "Reference" "C25"
+		(property "Reference" "C24"
 			(at 232.664 65.278 0)
 			(effects
@@
 			(project "tracker_pcb"
 				(path "/6aaa9514-f94e-4843-90d0-16960e4e49cb/856fce88-9666-4784-b480-ab1432c6ba59"
-					(reference "C25")
+					(reference "C24")
 					(unit 1)
 				)
@@
 		(on_board yes)
 		(dnp no)
-		(property "Reference" "R20"
+		(property "Reference" "R22"
 			(at 65.532 70.866 90)
 			(effects
@@
 			(project "tracker_pcb"
 				(path "/6aaa9514-f94e-4843-90d0-16960e4e49cb/856fce88-9666-4784-b480-ab1432c6ba59"
-					(reference "R20")
+					(reference "R22")
 					(unit 1)
 				)
@@
 		(dnp no)
 		(fields_autoplaced yes)
-		(property "Reference" "R24"
+		(property "Reference" "R26"
 			(at 147.32 90.1699 0)
 			(effects
@@
 			(project "tracker_pcb"
 				(path "/6aaa9514-f94e-4843-90d0-16960e4e49cb/856fce88-9666-4784-b480-ab1432c6ba59"
-					(reference "R24")
+					(reference "R26")
 					(unit 1)
 				)
@@
 		(on_board yes)
 		(dnp no)
-		(property "Reference" "C22"
+		(property "Reference" "C21"
 			(at 98.298 151.638 0)
 			(effects
@@
 			(project "tracker_pcb"
 				(path "/6aaa9514-f94e-4843-90d0-16960e4e49cb/856fce88-9666-4784-b480-ab1432c6ba59"
-					(reference "C22")
+					(reference "C21")
 					(unit 1)
 				)
@@
 		(on_board yes)
 		(dnp no)
-		(property "Reference" "C23"
+		(property "Reference" "C22"
 			(at 143.764 74.168 0)
 			(effects
@@
 			(project "tracker_pcb"
 				(path "/6aaa9514-f94e-4843-90d0-16960e4e49cb/856fce88-9666-4784-b480-ab1432c6ba59"
-					(reference "C23")
+					(reference "C22")
 					(unit 1)
 				)
@@
 		(on_board yes)
 		(dnp no)
-		(property "Reference" "C24"
+		(property "Reference" "C23"
 			(at 153.924 104.648 0)
 			(effects
@@
 			(project "tracker_pcb"
 				(path "/6aaa9514-f94e-4843-90d0-16960e4e49cb/856fce88-9666-4784-b480-ab1432c6ba59"
-					(reference "C24")
+					(reference "C23")
 					(unit 1)
 				)
@@
 		(on_board yes)
 		(dnp no)
-		(property "Reference" "R19"
+		(property "Reference" "R21"
 			(at 65.532 67.056 90)
 			(effects
@@
 			(project "tracker_pcb"
 				(path "/6aaa9514-f94e-4843-90d0-16960e4e49cb/856fce88-9666-4784-b480-ab1432c6ba59"
-					(reference "R19")
+					(reference "R21")
 					(unit 1)
 				)
@@
 		(dnp no)
 		(fields_autoplaced yes)
-		(property "Reference" "R23"
+		(property "Reference" "R25"
 			(at 137.16 60.9599 0)
 			(effects
@@
 			(project "tracker_pcb"
 				(path "/6aaa9514-f94e-4843-90d0-16960e4e49cb/856fce88-9666-4784-b480-ab1432c6ba59"
-					(reference "R23")
+					(reference "R25")
 					(unit 1)
 				)
@@
 		(dnp no)
 		(fields_autoplaced yes)
-		(property "Reference" "R25"
+		(property "Reference" "R27"
 			(at 156.21 81.28 90)
 			(effects
@@
 			(project "tracker_pcb"
 				(path "/6aaa9514-f94e-4843-90d0-16960e4e49cb/856fce88-9666-4784-b480-ab1432c6ba59"
-					(reference "R25")
+					(reference "R27")
 					(unit 1)
 				)
@@
 		(dnp no)
 		(fields_autoplaced yes)
-		(property "Reference" "J7"
+		(property "Reference" "J8"
 			(at 46.99 55.88 0)
 			(effects
@@
 			(project "tracker_pcb"
 				(path "/6aaa9514-f94e-4843-90d0-16960e4e49cb/856fce88-9666-4784-b480-ab1432c6ba59"
-					(reference "J7")
-					(unit 1)
-				)
+					(reference "J8")
+					(unit 1)
+				)

Commit message: SS changes
Parts:
- SW1, SW2: value SKRKAEE020 -> SKRKAHE020; LCSC C115357 -> C202388
Changed lines of the file:
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@@
 			)
 		)
-		(property "Value" "SKRKAEE020"
+		(property "Value" "SKRKAHE020"
 			(at 130.81 76.1999 90)
 			(effects
@@
 			)
 		)
-		(property "LCSC" "C115357"
+		(property "LCSC" "C202388"
 			(at 130.81 73.6599 0)
 			(effects
@@
 			)
 		)
-		(property "Value" "SKRKAEE020"
+		(property "Value" "SKRKAHE020"
 			(at 140.97 106.6799 90)
 			(effects
@@
 			)
 		)
-		(property "LCSC" "C115357"
+		(property "LCSC" "C202388"
 			(at 140.97 104.1399 0)
 			(effects

Commit message: add 3pin jst for analog
Connections:
- net IO8: now reaches R27.1, U11.22 (IO8)

Commit message: update BOM
Parts:
- J8: value USB_C_Receptacle_USB2.0_16P -> TYPE-C-31-M-12; LCSC C5184243 -> C165948
- SW1, SW2: LCSC C202388 -> C493285
Changed lines of the file:
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@@
 			)
 		)
-		(property "LCSC" "C202388"
+		(property "LCSC" "C493285"
 			(at 130.81 73.6599 0)
 			(effects
@@
 			)
 		)
-		(property "Value" "USB_C_Receptacle_USB2.0_16P"
+		(property "Value" "TYPE-C-31-M-12"
 			(at 46.99 58.42 0)
 			(effects
@@
 			)
 		)
-		(property "Datasheet" "https://www.usb.org/sites/default/files/documents/usb_type-c.zip"
+		(property "Datasheet" "https://jlcpcb.com/api/file/downloadByFileSystemAccessId/8550723676069908480"
 			(at 50.8 78.74 0)
 			(effects
@@
 			)
 		)
-		(property "LCSC" "C5184243"
+		(property "LCSC" "C165948"
 			(at 46.99 55.88 0)
 			(effects
@@
 			)
 		)
-		(property "LCSC" "C202388"
+		(property "LCSC" "C493285"
 			(at 140.97 104.1399 0)
 			(effects

Commit message: v2 hardware changes
Parts:
- added C22: 100nF, Capacitor_SMD:C_0603_1608Metric, symbol Device:C
- added R27, R28: 10k, Resistor_SMD:R_0603_1608Metric, symbol Device:R_US
- added U9: SN74AUP2G125YZPR, footprint:YZP8, symbol symbol:SN74AUP2G125YZPR
- renumbered C21 to C23, C22 to C24, C23 to C25, C24 to C26, J8 to J9, R21 to R23, R22 to R24, R23 to R25, R24 to R26, R25 to R29, R26 to R30, R27 to R31, U9 to U10, U10 to U11, U11 to U12
Connections:
- net GND: now also C22.2, R27.1, R28.1, U9.D1 (GND)
- net IO6: now also U9.B1 (1A); no longer U11.A1 (A)
- net IO7: now also U9.D2 (2A); no longer U11.B1 (B)
- net IO8: now also U9.A1 (~{1OE}), U9.B2 (~{2OE})
- net V33: now also C22.1, U9.A2 (VCC)
- new net: R28.2, U11.B1 (B), U9.C1 (2Y)
- new net: R27.2, U11.A1 (A), U9.C2 (1Y)
Other:
- note added: "CSMUX_A"
- note added: "CSMUX_B"
- note added: "SPI_CSS"
- moved on the sheet: C23
