File: hardware/tracker_pcb/esp32.kicad_sch (KiCad schematic)
At the start: 21 parts, among them J9 TYPE-C-31-M-12, SW1 SKRKAHE020, SW2 SKRKAHE020, U10 USBLC6-2SC6, U11 SN74LVC1G139, U12 ESP32-C6-MINI-1U-N4, U9 SN74AUP2G125YZPR

Commit message: more motor safety
Parts:
- removed C22: 100nF, Capacitor_SMD:C_0603_1608Metric, symbol Device:C
- removed R27, R28: 10k, Resistor_SMD:R_0603_1608Metric, symbol Device:R_US
- removed U11: SN74LVC1G139, footprint:BGA8C50P2X4_89X189X50, symbol symbol:SN74LVC1G139
- removed U9: SN74AUP2G125YZPR, footprint:YZP8, symbol symbol:SN74AUP2G125YZPR
- added U7: SN74AHC138RGYR, footprint:RGY16_2P55X2P05, symbol symbol:SN74AHC138RGYR
- renumbered C23 to C21, C24 to C22, C25 to C23, C26 to C24, R29 to R27, R30 to R28, R31 to R29, U10 to U8, U12 to U9
Connections:
- net GND: now also U7.17 (EPAD), U7.3 (C), U7.5 (~{G2B}), U7.8 (GND)
- net IO6: now also U7.1 (A)
- net IO7: now also U7.2 (B)
- net IO8: now also U7.4 (~{G2A})
- net NSS_CS0: now also U7.15 (~{Y0})
- net NSS_CS1: now also U7.14 (~{Y1})
- net NSS_CS2: now also U7.13 (~{Y2})
- net NSS_CS3: now also U7.12 (~{Y3})
- net V33: now also U7.16 (VCC), U7.6 (G1)
- no-connect marks 2 -> 6
Other:
- note added: "CS MUX"
- note added: "SPI_CS"
- note removed: "CSMUX_A"
- note removed: "CSMUX_B"
- note removed: "SPI_CSS"
- moved on the sheet: C21
