File: hardware/tracker_pcb/iso-input.kicad_sch (KiCad schematic)
At the start: 5 parts, among them Q1 LTV-817S-TA1-D

Commit message: Add zener diodes to properly bias optos across 6-35V input rnge
Parts:
- added D9: DFLZ107, footprint:DFLZ107, symbol Device:D_Zener
- D5: value 1N4148W(SOD-123) -> 1N4148W
- LED1: value C72039 -> GRNLED
- R13: value 1.8k -> 1.2k; footprint Resistor_SMD:R_0805_2012Metric_Pad1.20x1.40mm_HandSolder -> Resistor_SMD:R_2010_5025Metric; LCSC C17513 -> C17398
Connections:
- net IN-: now also D9.2 (A)
- net at D5.1 (K), LED1.2 (A), R13.2: now also D9.1 (K)
Changed lines of the file:
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@@
+	)
+	(junction
+		(at 114.3 85.09)
+		(diameter 0)
+		(color 0 0 0 0)
 	)
 	(junction
@@
 	)
 	(junction
+		(at 114.3 97.79)
+		(diameter 0)
+		(color 0 0 0 0)
+	)
+	(junction
 		(at 127 85.09)
 		(diameter 0)
@@
 	(wire
 		(pts
+			(xy 114.3 97.79) (xy 127 97.79)
+		)
+		(stroke
+			(width 0)
+			(type default)
+		)
+	)
+	(wire
+		(pts
+			(xy 114.3 85.09) (xy 114.3 87.63)
+		)
+		(stroke
+			(width 0)
+			(type default)
+		)
+	)
+	(wire
+		(pts
 			(xy 139.7 85.09) (xy 146.05 85.09)
 		)
@@
 	(wire
 		(pts
-			(xy 90.17 97.79) (xy 127 97.79)
+			(xy 90.17 97.79) (xy 114.3 97.79)
 		)
 		(stroke
@@
 	(wire
 		(pts
-			(xy 110.49 85.09) (xy 127 85.09)
+			(xy 110.49 85.09) (xy 114.3 85.09)
+		)
+		(stroke
+			(width 0)
+			(type default)
+		)
+	)
+	(wire
+		(pts
+			(xy 114.3 95.25) (xy 114.3 97.79)
 		)
 		(stroke
@@
 		(pts
 			(xy 127 95.25) (xy 127 97.79)
+		)
+		(stroke
+			(width 0)
+			(type default)
+		)
+	)
+	(wire
+		(pts
+			(xy 114.3 85.09) (xy 127 85.09)
 		)
 		(stroke
@@
 			)
 		)
-		(property "Value" "C72039"
-			(at 128.905 88.265 0)
+		(property "Value" "GRNLED"
+			(at 137.16 86.614 0)
 			(effects
 				(font
@@
 			)
 		)
-		(property "Value" "1.8k"
+		(property "Value" "1.2k"
 			(at 106.68 81.28 90)
 			(effects
@@
 			)
 		)
-		(property "Footprint" "Resistor_SMD:R_0805_2012Metric_Pad1.20x1.40mm_HandSolder"
+		(property "Footprint" "Resistor_SMD:R_2010_5025Metric"
 			(at 106.934 84.074 90)
 			(effects
@@
 			)
 		)
-		(property "LCSC" "C17513"
+		(property "LCSC" "C17398 "
 			(at 106.68 78.74 0)
 			(effects
@@
 				(path "/6aaa9514-f94e-4843-90d0-16960e4e49cb/b128d80c-4aa3-4c05-bd4f-543db8edd72e"
 					(reference "R17")
+					(unit 1)
+				)
+			)
+		)
+	)
+	(symbol
+		(lib_id "Device:D_Zener")
+		(at 114.3 91.44 270)
+		(unit 1)
+		(exclude_from_sim no)
+		(in_bom yes)
+		(on_board yes)
+		(dnp no)
+		(fields_autoplaced yes)
+		(property "Reference" "D9"
+			(at 116.84 90.1699 90)
+			(effects
+				(font
+					(size 1.27 1.27)
+				)
+				(justify left)
+			)
+		)
+		(property "Value" "DFLZ107"
+			(at 116.84 92.7099 90)
+			(effects
+				(font
+					(size 1.27 1.27)
+				)
+				(justify left)
+			)
+		)
+		(property "Footprint" "footprint:DFLZ107"
+			(at 114.3 91.44 0)
+			(effects
+				(font
+					(size 1.27 1.27)
+				)
+				(hide yes)
+			)
+		)
+		(property "Datasheet" "~"
+			(at 114.3 91.44 0)
+			(effects
+				(font
+					(size 1.27 1.27)
+				)
+				(hide yes)
+			)
+		)
+		(property "Description" "Zener diode"
+			(at 114.3 91.44 0)
+			(effects
+				(font
+					(size 1.27 1.27)
+				)
+				(hide yes)
+			)
+		)
+		(pin "1"
+		)
+		(pin "2"
+		)
+		(instances
+			(project ""
+				(path "/6aaa9514-f94e-4843-90d0-16960e4e49cb/04328898-976a-48a2-86bf-9938cb4aefd5"
+					(reference "D10")
+					(unit 1)
+				)
+				(path "/6aaa9514-f94e-4843-90d0-16960e4e49cb/45a2292e-2f51-4a4c-a627-74180fb6fdfe"
+					(reference "D12")
+					(unit 1)
+				)
+				(path "/6aaa9514-f94e-4843-90d0-16960e4e49cb/45c78875-26ba-4b22-bc82-79a51b704824"
+					(reference "D9")
+					(unit 1)
+				)
+				(path "/6aaa9514-f94e-4843-90d0-16960e4e49cb/b128d80c-4aa3-4c05-bd4f-543db8edd72e"
+					(reference "D11")
 					(unit 1)
 				)
@@
 			)
 		)
-		(property "Value" "1N4148W(SOD-123)"
-			(at 105.664 93.98 90)
-			(effects
-				(font
+		(property "Value" "1N4148W"
+			(at 129.032 91.44 90)
+			(effects
+				(font

Commit message: SS changes
Parts:
- R13: LCSC C17398 -> C2078103
Changed lines of the file:
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@@
 			)
 		)
-		(property "LCSC" "C17398 "
+		(property "LCSC" "C2078103"
 			(at 106.68 78.74 0)
 			(effects

Commit message: add 3pin jst for analog
Parts:
- D5: renamed from D9; value DFLZ107 -> DFLZ10-7; LCSC (none) -> C151371; LCSC Part Name (none) -> DFLZ10-7
- renumbered D5 to D6

Commit message: v2 hardware changes
Parts:
- renumbered D5 to D7, D6 to D8, R13 to R15, R14 to R16
Changed lines of the file:
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@@
 		(dnp no)
 		(fields_autoplaced yes)
-		(property "Reference" "R13"
+		(property "Reference" "R15"
 			(at 106.68 78.74 90)
 			(effects
@@
 			(project "tracker_pcb"
 				(path "/6aaa9514-f94e-4843-90d0-16960e4e49cb/04328898-976a-48a2-86bf-9938cb4aefd5"
+					(reference "R17")
+					(unit 1)
+				)
+				(path "/6aaa9514-f94e-4843-90d0-16960e4e49cb/45a2292e-2f51-4a4c-a627-74180fb6fdfe"
+					(reference "R21")
+					(unit 1)
+				)
+				(path "/6aaa9514-f94e-4843-90d0-16960e4e49cb/45c78875-26ba-4b22-bc82-79a51b704824"
 					(reference "R15")
 					(unit 1)
 				)
-				(path "/6aaa9514-f94e-4843-90d0-16960e4e49cb/45a2292e-2f51-4a4c-a627-74180fb6fdfe"
+				(path "/6aaa9514-f94e-4843-90d0-16960e4e49cb/b128d80c-4aa3-4c05-bd4f-543db8edd72e"
 					(reference "R19")
-					(unit 1)
-				)
-				(path "/6aaa9514-f94e-4843-90d0-16960e4e49cb/45c78875-26ba-4b22-bc82-79a51b704824"
-					(reference "R13")
-					(unit 1)
-				)
-				(path "/6aaa9514-f94e-4843-90d0-16960e4e49cb/b128d80c-4aa3-4c05-bd4f-543db8edd72e"
-					(reference "R17")
 					(unit 1)
 				)
@@
 		(dnp no)
 		(fields_autoplaced yes)
-		(property "Reference" "D5"
+		(property "Reference" "D7"
 			(at 116.84 90.1699 90)
 			(effects
@@
 			(project ""
 				(path "/6aaa9514-f94e-4843-90d0-16960e4e49cb/04328898-976a-48a2-86bf-9938cb4aefd5"
+					(reference "D9")
+					(unit 1)
+				)
+				(path "/6aaa9514-f94e-4843-90d0-16960e4e49cb/45a2292e-2f51-4a4c-a627-74180fb6fdfe"
+					(reference "D13")
+					(unit 1)
+				)
+				(path "/6aaa9514-f94e-4843-90d0-16960e4e49cb/45c78875-26ba-4b22-bc82-79a51b704824"
 					(reference "D7")
 					(unit 1)
 				)
-				(path "/6aaa9514-f94e-4843-90d0-16960e4e49cb/45a2292e-2f51-4a4c-a627-74180fb6fdfe"
+				(path "/6aaa9514-f94e-4843-90d0-16960e4e49cb/b128d80c-4aa3-4c05-bd4f-543db8edd72e"
 					(reference "D11")
-					(unit 1)
-				)
-				(path "/6aaa9514-f94e-4843-90d0-16960e4e49cb/45c78875-26ba-4b22-bc82-79a51b704824"
-					(reference "D5")
-					(unit 1)
-				)
-				(path "/6aaa9514-f94e-4843-90d0-16960e4e49cb/b128d80c-4aa3-4c05-bd4f-543db8edd72e"
-					(reference "D9")
 					(unit 1)
 				)
@@
 		(on_board yes)
 		(dnp no)
-		(property "Reference" "#PWR018"
+		(property "Reference" "#PWR019"
 			(at 173.99 104.14 0)
 			(effects
@@
 			(project "tracker_pcb"
 				(path "/6aaa9514-f94e-4843-90d0-16960e4e49cb/04328898-976a-48a2-86bf-9938cb4aefd5"
+					(reference "#PWR020")
+					(unit 1)
+				)
+				(path "/6aaa9514-f94e-4843-90d0-16960e4e49cb/45a2292e-2f51-4a4c-a627-74180fb6fdfe"
+					(reference "#PWR022")
+					(unit 1)
+				)
+				(path "/6aaa9514-f94e-4843-90d0-16960e4e49cb/45c78875-26ba-4b22-bc82-79a51b704824"
 					(reference "#PWR019")
 					(unit 1)
 				)
-				(path "/6aaa9514-f94e-4843-90d0-16960e4e49cb/45a2292e-2f51-4a4c-a627-74180fb6fdfe"
+				(path "/6aaa9514-f94e-4843-90d0-16960e4e49cb/b128d80c-4aa3-4c05-bd4f-543db8edd72e"
 					(reference "#PWR021")
-					(unit 1)
-				)
-				(path "/6aaa9514-f94e-4843-90d0-16960e4e49cb/45c78875-26ba-4b22-bc82-79a51b704824"
-					(reference "#PWR018")
-					(unit 1)
-				)
-				(path "/6aaa9514-f94e-4843-90d0-16960e4e49cb/b128d80c-4aa3-4c05-bd4f-543db8edd72e"
-					(reference "#PWR020")
 					(unit 1)
 				)
@@
 		(dnp no)
 		(fields_autoplaced yes)
-		(property "Reference" "R14"
+		(property "Reference" "R16"
 			(at 181.61 73.6599 0)
 			(effects
@@
 			(project "tracker_pcb"
 				(path "/6aaa9514-f94e-4843-90d0-16960e4e49cb/04328898-976a-48a2-86bf-9938cb4aefd5"
+					(reference "R18")
+					(unit 1)
+				)
+				(path "/6aaa9514-f94e-4843-90d0-16960e4e49cb/45a2292e-2f51-4a4c-a627-74180fb6fdfe"
+					(reference "R22")
+					(unit 1)
+				)
+				(path "/6aaa9514-f94e-4843-90d0-16960e4e49cb/45c78875-26ba-4b22-bc82-79a51b704824"
 					(reference "R16")
 					(unit 1)
 				)
-				(path "/6aaa9514-f94e-4843-90d0-16960e4e49cb/45a2292e-2f51-4a4c-a627-74180fb6fdfe"
+				(path "/6aaa9514-f94e-4843-90d0-16960e4e49cb/b128d80c-4aa3-4c05-bd4f-543db8edd72e"
 					(reference "R20")
-					(unit 1)
-				)
-				(path "/6aaa9514-f94e-4843-90d0-16960e4e49cb/45c78875-26ba-4b22-bc82-79a51b704824"
-					(reference "R14")
-					(unit 1)
-				)
-				(path "/6aaa9514-f94e-4843-90d0-16960e4e49cb/b128d80c-4aa3-4c05-bd4f-543db8edd72e"
-					(reference "R18")
 					(unit 1)
 				)
@@
 		(on_board yes)
 		(dnp no)
-		(property "Reference" "D6"
+		(property "Reference" "D8"
 			(at 125.73 86.36 90)
 			(effects
@@
 			(project "tracker_pcb"
 				(path "/6aaa9514-f94e-4843-90d0-16960e4e49cb/04328898-976a-48a2-86bf-9938cb4aefd5"
+					(reference "D10")
+					(unit 1)
+				)
+				(path "/6aaa9514-f94e-4843-90d0-16960e4e49cb/45a2292e-2f51-4a4c-a627-74180fb6fdfe"
+					(reference "D14")
+					(unit 1)
+				)
+				(path "/6aaa9514-f94e-4843-90d0-16960e4e49cb/45c78875-26ba-4b22-bc82-79a51b704824"
 					(reference "D8")
 					(unit 1)
 				)
-				(path "/6aaa9514-f94e-4843-90d0-16960e4e49cb/45a2292e-2f51-4a4c-a627-74180fb6fdfe"
+				(path "/6aaa9514-f94e-4843-90d0-16960e4e49cb/b128d80c-4aa3-4c05-bd4f-543db8edd72e"
 					(reference "D12")
 					(unit 1)
 				)
-				(path "/6aaa9514-f94e-4843-90d0-16960e4e49cb/45c78875-26ba-4b22-bc82-79a51b704824"
-					(reference "D6")
-					(unit 1)
-				)
-				(path "/6aaa9514-f94e-4843-90d0-16960e4e49cb/b128d80c-4aa3-4c05-bd4f-543db8edd72e"
-					(reference "D10")
-					(unit 1)
-				)
